Commit message: added URDF for core robot

File: description/robot_core.xacro (robot description, xacro)
@@ -40,4 +40,7 @@
         </xacro:inertial_box>
     </link>
+    <gazebo reference='chassis_link'>
+        <material>Gazebo/White</material>
+    </gazebo>
     <!-- LEFT WHEEL LINK -->
     <joint name="left_wheel_joint" type="continuous">
@@ -63,4 +66,7 @@
         </xacro:inertial_cylinder>
     </link>
+    <gazebo reference='left_wheel_link'>
+        <material>Gazebo/Blue</material>
+    </gazebo>
     <!-- RIGHT WHEEL LINK -->
     <joint name="right_wheel_joint" type="continuous">
@@ -86,4 +92,7 @@
         </xacro:inertial_cylinder>
     </link>
+    <gazebo reference='right_wheel_link'>
+        <material>Gazebo/Blue</material>
+    </gazebo>
     <!-- CASTER WHEEL LINK -->
     <joint name="caster_wheel_join" type="fixed">
@@ -108,3 +117,8 @@
         </xacro:inertial_sphere>
     </link>
+    <gazebo reference='caster_wheel_link'>
+        <material>Gazebo/Orange</material>
+        <mu1 value='0.001'/>
+        <mu2 value='0.001'/>
+    </gazebo>
 </robot>
